File: project-hw-2-18650.kicad_pcb (KiCad board)
At the start: 2 copper layers, 98 x 44 mm, 22 parts, among them J1 2060-452_998-404, Q1 Q_Toshiba_SSM3J328R, SW1 PTS810_SJM_250_SMTR_LFS, U1 TPS62933, U2 TPS259630

Commit message: Add clarity to the choice resistors
Parts:
- R3: value 31.6k -> UVLO-R1
- R4: value 7.5k -> UVLO-R2
- R5: value 470 -> Current limit
Other:
- board text added: "Current limit 470: 1.93A 1k: 0.91A 7.5k: 132mA"
- board text added: "EN/UVLO R1: 100k R2: 22k Cutoff: 6.1V Quiescent current: 61uA R1: 47k R2: 10.5k Cutoff: 6.024V Quiescent current: R1: 56k R2: 12.7k Cutoff: 5.95V Quiescent current:"
- board text added: "Vchoice 52.3k = 5V 31.6k = 3.328V"
Changed lines of the file:
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@@
 			)
 		)
-		(property "Value" "31.6k"
-			(at 0 -1.5 -90)
+		(property "Value" "UVLO-R1"
+			(at -2.1 -3.6 45)
 			(layer "F.Fab")
 			(effects
@@
 		)
 		(property "Value" "10k"
-			(at 3.7 0.05 0)
+			(at 2.6 0.05 0)
 			(layer "F.Fab")
 			(effects
@@
 		)
 		(property "Value" "6.8uH"
-			(at -0.2 -4.1 -90)
+			(at -0.2 -4.1 90)
 			(unlocked yes)
 			(layer "F.Fab")
@@
 			)
 		)
-		(property "Value" "7.5k"
-			(at 0.6 -1.5 90)
+		(property "Value" "UVLO-R2"
+			(at 0.1 -4.4 180)
 			(layer "F.Fab")
 			(effects
@@
 			)
 		)
-		(property "Value" "470"
-			(at -2.9 0 90)
+		(property "Value" "Current limit"
+			(at -0.7 -0.9 90)
 			(layer "F.Fab")
+			(hide yes)
 			(effects
 				(font
@@
 		)
 	)
+	(gr_text "EN/UVLO\n\nR1: 100k\nR2: 22k\nCutoff: 6.1V\nQuiescent current: 61uA\n\nR1: 47k\nR2: 10.5k\nCutoff: 6.024V\nQuiescent current: \n\nR1: 56k\nR2: 12.7k\nCutoff: 5.95V\nQuiescent current: "
+		(at 21 101 0)
+		(layer "F.Fab")
+		(effects
+			(font
+				(size 1.5 1.5)
+				(thickness 0.3)
+				(bold yes)
+			)
+			(justify left bottom)
+		)
+	)
+	(gr_text "Current limit\n\n470: 1.93A\n1k: 0.91A\n7.5k: 132mA"
+		(at 57 74 0)
+		(layer "F.Fab")
+		(effects
+			(font
+				(size 1.5 1.5)
+				(thickness 0.3)
+				(bold yes)
+			)
+			(justify left bottom)
+		)
+	)
+	(gr_text "Vchoice\n\n52.3k = 5V\n31.6k = 3.328V"
+		(at 81 71 0)
+		(layer "F.Fab")
+		(effects
+			(font
+				(size 1.5 1.5)
+				(thickness 0.3)
+				(bold yes)
+			)
+			(justify left bottom)
+		)
+	)

Commit message: Add max input voltage information
Other:
- board text added: "Max input voltage: - 19V eFuse - 20V P-MOSFET"
Changed lines of the file:
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@@
+		)
+	)
+	(gr_text "Max input voltage:\n- 19V eFuse\n- 20V P-MOSFET"
+		(at 57 88 0)
+		(layer "F.Fab")
+		(effects
+			(font
+				(size 1.5 1.5)
+				(thickness 0.3)
+				(bold yes)
+			)
+			(justify left bottom)
 		)
 	)
